File: kicad/TranspOtterNG.kicad_pcb (KiCad board)
At the start: 2 copper layers, 100 x 45 mm, 64 parts, among them J1 UART/I2C, J2 UART/IO/ANALOG, J3 Conn_01x04_Male, J4 GameTrak, J7 xt30, J8 Conn_01x05_Male, J9 Conn_01x16_Female, P1 CONN_WII, Q1 Q_NMOS_GDS, Q2 Q_PMOS_GDS, SW1 Flash, SW2 Reset, U1 AMS1117, U2 URB4805YMD-6WR3, U3 RFM69HCW, U4 ESP-12E, U5 PCF8574

Commit message: minor changes
Parts:
- moved R26 10.2 mm to (165.0, 46.2), turned to 90 degrees
- moved R18 5.20 mm to (135.2, 45.5)
- moved R22 5.20 mm to (139.2, 47.0)
- moved R27 5.20 mm to (132.9, 48.6)
- moved R28 5.20 mm to (132.9, 45.5)
- moved R19 5.20 mm to (135.1, 47.0)
- moved R20 5.20 mm to (135.1, 48.5)
- moved R21 5.20 mm to (139.1, 45.5)
- moved R23 5.20 mm to (139.1, 48.5)
- moved J9 5.00 mm to (125.6, 42.5)
- moved U5 4.90 mm to (155.9, 50.1)
- moved C10 4.61 mm to (162.8, 46.2)
- moved C1 1.90 mm to (162.9, 49.6)
- moved C13 1.90 mm to (165.4, 50.8)
- moved R11 1.90 mm to (162.9, 52.5)
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Connections:
- C5 pad 1: TX0_SCL -> Net-(C5-Pad1)
- C6 pad 1: TX1_ADC1 -> Net-(C6-Pad1)
- C7 pad 1: RX0_SDA -> Net-(C7-Pad1)
- C8 pad 1: RX1_ADC2 -> Net-(C8-Pad1)
- J1 pad 2: Net-(J1-Pad2) -> Net-(C5-Pad1)
- J1 pad 3: Net-(J1-Pad3) -> Net-(C7-Pad1)
- J2 pad 2: Net-(J2-Pad2) -> Net-(C6-Pad1)
- J2 pad 3: Net-(J2-Pad3) -> Net-(C8-Pad1)
- R4 pad 2: Net-(J1-Pad2) -> Net-(C5-Pad1)
- R5 pad 2: Net-(J1-Pad3) -> Net-(C7-Pad1)
- R6 pad 2: Net-(J2-Pad2) -> Net-(C6-Pad1)
- R7 pad 2: Net-(J2-Pad3) -> Net-(C8-Pad1)
Routing:
- net LED_K: track 13.5 -> 3.45 mm
- net +5V: track 111.3 -> 103.6 mm
- net CS: track 17.1 -> 23.5 mm, vias 0 -> 1
- net Net-(C5-Pad1): track 0.00 -> 6.15 mm
- net Net-(C8-Pad1): track 0.00 -> 5.55 mm
- net Net-(C6-Pad1): track 0.00 -> 5.55 mm
- net Net-(C7-Pad1): track 0.00 -> 5.48 mm
- net Net-(J1-Pad2): track 4.61 -> 0.00 mm
- net TX0_SCL: track 79.6 -> 83.8 mm
- net Net-(J1-Pad3): track 4.23 -> 0.00 mm
- net Net-(J2-Pad2): track 4.10 -> 0.00 mm
- net Net-(J2-Pad3): track 4.08 -> 0.00 mm
- net RX0_SDA: track 91.3 -> 94.9 mm
- net GPIO4: track 21.3 -> 23.3 mm
- net RW: track 20.8 -> 18.9 mm
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Other:
- outline, holes or cut-outs redrawn
