File: kicad/TranspOtterNG.sch (KiCad schematic (older format))
At the start: 31 parts, among them J1 UART/I2C, J2 UART/IO/ANALOG, J3 Display, J4 GameTrak, J6 Nunchuk, J7 VCC, U1 AMS1117

Commit message: added stepdown
Parts:
- removed C1: 1u, Capacitors_SMD:C_0805, symbol Device:C_Small
- added C10, C11: 100n, Capacitors_SMD:C_0603, symbol Device:C_Small
- added C12, C9: 470u, Capacitors_SMD:CP_Elec_5x5.3, symbol Device:CP_Small
- added D4: 1N5822, Diodes_SMD:D_SMA, symbol Diode:1N5822
- added L1: L, Inductors_SMD:L_Taiyo-Yuden_MD-5050, symbol Device:L
- added U2: LM2596S-5, TO_SOT_Packages_SMD:TO-263-5_TabPin3, symbol Regulator_Switching:LM2596S-5
Connections:
- net labels added: +5V
- wire segments 45 -> 53
Other:
- note added: "5V\n"
Changed lines of the file:
@@
 Connection ~ 5350 1200
-$Comp
-L power:+15V #PWR0105
-U 1 1 5BA38B61
-P 4000 1200
-F 0 "#PWR0105" H 4000 1050 50  0001 C CNN
-F 1 "+15V" H 4015 1373 50  0000 C CNN
-F 2 "" H 4000 1200 50  0001 C CNN
-F 3 "" H 4000 1200 50  0001 C CNN
-	1    4000 1200
-	1    0    0    -1
-$EndComp
 $Comp
 L power:VCC #PWR0106
@@
 F 3 "" H 5750 1200 50  0001 C CNN
 	1    5750 1200
-	1    0    0    -1
-$EndComp
-$Comp
-L power:GND #PWR0107
-U 1 1 5BA38BF0
-P 4050 1400
-F 0 "#PWR0107" H 4050 1150 50  0001 C CNN
-F 1 "GND" H 4055 1227 50  0000 C CNN
-F 2 "" H 4050 1400 50  0001 C CNN
-F 3 "" H 4050 1400 50  0001 C CNN
-	1    4050 1400
 	1    0    0    -1
 $EndComp
@@
 	7700 600  7700 2200
 Wire Wire Line
-	4000 1200 4050 1200
-$Comp
-L Device:C_Small C1
-U 1 1 5BA3BD0F
-P 4050 1300
-F 0 "C1" H 4142 1346 50  0000 L CNN
-F 1 "1u" H 4142 1255 50  0000 L CNN
-F 2 "Capacitors_SMD:C_0805" H 4050 1300 50  0001 C CNN
-F 3 "~" H 4050 1300 50  0001 C CNN
-	1    4050 1300
-	1    0    0    -1
-$EndComp
-Connection ~ 4050 1200
-Wire Wire Line
-	4050 1200 4400 1200
-Wire Wire Line
 	5350 1200 5700 1200
 $Comp
@@
 Wire Wire Line
 	5700 1200 5750 1200
-Wire Notes Line
-	600  600  7700 600
-Wire Notes Line
-	600  2200 7700 2200
 $Comp
 L Device:R R4
@@
 Wire Wire Line
 	3550 2650 3900 2650
+$Comp
+L Regulator_Switching:LM2596S-5 U2
+U 1 1 5BA3B38B
+P 9300 1450
+F 0 "U2" H 9300 1817 50  0000 C CNN
+F 1 "LM2596S-5" H 9300 1726 50  0000 C CNN
+F 2 "TO_SOT_Packages_SMD:TO-263-5_TabPin3" H 9350 1200 50  0001 L CIN
+F 3 "http://www.ti.com/lit/ds/symlink/lm2596.pdf" H 9300 1450 50  0001 C CNN
+	1    9300 1450
+	1    0    0    -1
+$EndComp
+$Comp
+L Device:C_Small C10
+U 1 1 5BA3B7B8
+P 8400 1450
+F 0 "C10" H 8492 1496 50  0000 L CNN
+F 1 "100n" H 8492 1405 50  0000 L CNN
+F 2 "Capacitors_SMD:C_0603" H 8400 1450 50  0001 C CNN
+F 3 "~" H 8400 1450 50  0001 C CNN
+	1    8400 1450
+	1    0    0    -1
+$EndComp
+$Comp
+L power:+15V #PWR0105
+U 1 1 5BA3B7C1
+P 8000 1350
+F 0 "#PWR0105" H 8000 1200 50  0001 C CNN
+F 1 "+15V" H 8015 1523 50  0000 C CNN
+F 2 "" H 8000 1350 50  0001 C CNN
+F 3 "" H 8000 1350 50  0001 C CNN
+	1    8000 1350
+	1    0    0    -1
+$EndComp
+$Comp
+L power:GND #PWR0123
+U 1 1 5BA3B7C7
+P 8050 1550
+F 0 "#PWR0123" H 8050 1300 50  0001 C CNN
+F 1 "GND" H 8055 1377 50  0000 C CNN
+F 2 "" H 8050 1550 50  0001 C CNN
+F 3 "" H 8050 1550 50  0001 C CNN
+	1    8050 1550
+	1    0    0    -1
+$EndComp
+$Comp
+L power:GND #PWR0131
+U 1 1 5BA3B7CD
+P 8400 1550
+F 0 "#PWR0131" H 8400 1300 50  0001 C CNN
+F 1 "GND" H 8405 1377 50  0000 C CNN
+F 2 "" H 8400 1550 50  0001 C CNN
+F 3 "" H 8400 1550 50  0001 C CNN
+	1    8400 1550
+	1    0    0    -1
+$EndComp
+$Comp
+L power:+5V #PWR0132
+U 1 1 5BA3C54C
+P 4000 1200
+F 0 "#PWR0132" H 4000 1050 50  0001 C CNN
+F 1 "+5V" H 4015 1373 50  0000 C CNN
+F 2 "" H 4000 1200 50  0001 C CNN
+F 3 "" H 4000 1200 50  0001 C CNN
+	1    4000 1200
+	1    0    0    -1
+$EndComp
+$Comp
+L Device:CP_Small C9
+U 1 1 5BA3C822
+P 8050 1450
+F 0 "C9" H 8138 1496 50  0000 L CNN
+F 1 "470u" H 8138 1405 50  0000 L CNN
+F 2 "Capacitors_SMD:CP_Elec_5x5.3" H 8050 1450 50  0001 C CNN
+F 3 "~" H 8050 1450 50  0001 C CNN
+	1    8050 1450
+	1    0    0    -1
+$EndComp
+$Comp
+L power:GND #PWR0133
+U 1 1 5BA3D885
+P 8800 1550
+F 0 "#PWR0133" H 8800 1300 50  0001 C CNN
+F 1 "GND" H 8805 1377 50  0000 C CNN
+F 2 "" H 8800 1550 50  0001 C CNN
+F 3 "" H 8800 1550 50  0001 C CNN
+	1    8800 1550
+	1    0    0    -1
+$EndComp
+$Comp
+L power:GND #PWR0134
+U 1 1 5BA3D90D
+P 9300 1750
+F 0 "#PWR0134" H 9300 1500 50  0001 C CNN
+F 1 "GND" H 9305 1577 50  0000 C CNN
+F 2 "" H 9300 1750 50  0001 C CNN
+F 3 "" H 9300 1750 50  0001 C CNN
+	1    9300 1750
+	1    0    0    -1
+$EndComp
+$Comp
+L Diode:1N5822 D4
+U 1 1 5BA3DAF0
+P 9900 1700
+F 0 "D4" V 9854 1779 50  0000 L CNN
+F 1 "1N5822" V 9945 1779 50  0000 L CNN
+F 2 "Diodes_SMD:D_SMA" H 9900 1525 50  0001 C CNN
+F 3 "http://www.vishay.com/docs/88526/1n5820.pdf" H 9900 1700 50  0001 C CNN
+	1    9900 1700
+	0    1    1    0
+$EndComp
+$Comp
+L Device:L L1
+U 1 1 5BA3DC35
+P 10150 1550
+F 0 "L1" V 10340 1550 50  0000 C CNN
+F 1 "L" V 10249 1550 50  0000 C CNN
+F 2 "Inductors_SMD:L_Taiyo-Yuden_MD-5050" H 10150 1550 50  0001 C CNN
+F 3 "~" H 10150 1550 50  0001 C CNN
+	1    10150 1550
+	0    -1   -1   0
+$EndComp
+Wire Wire Line
+	8400 1350 8800 1350
+Connection ~ 8050 1350
+Wire Wire Line
+	8050 1350 8400 1350
+Wire Wire Line
+	8000 1350 8050 1350
+Connection ~ 8400 1350
+$Comp
+L Device:C_Small C11
+U 1 1 5BA3EBE8
+P 10400 1650
+F 0 "C11" H 10492 1696 50  0000 L CNN
+F 1 "100n" H 10492 1605 50  0000 L CNN
+F 2 "Capacitors_SMD:C_0603" H 10400 1650 50  0001 C CNN
+F 3 "~" H 10400 1650 50  0001 C CNN
+	1    10400 1650
+	1    0    0    -1
+$EndComp
+$Comp
+L power:GND #PWR0135
+U 1 1 5BA3EBEF
+P 10750 1750
+F 0 "#PWR0135" H 10750 1500 50  0001 C CNN
+F 1 "GND" H 10755 1577 50  0000 C CNN
+F 2 "" H 10750 1750 50  0001 C CNN
+F 3 "" H 10750 1750 50  0001 C CNN
+	1    10750 1750
+	1    0    0    -1
+$EndComp
+$Comp
+L power:GND #PWR0136
+U 1 1 5BA3EBF5
+P 10400 1750
+F 0 "#PWR0136" H 10400 1500 50  0001 C CNN
+F 1 "GND" H 10405 1577 50  0000 C CNN
+F 2 "" H 10400 1750 50  0001 C CNN
+F 3 "" H 10400 1750 50  0001 C CNN
+	1    10400 1750
+	1    0    0    -1
+$EndComp
+$Comp
+L Device:CP_Small C12
+U 1 1 5BA3EBFB
+P 10750 1650
+F 0 "C12" H 10838 1696 50  0000 L CNN
+F 1 "470u" H 10838 1605 50  0000 L CNN
+F 2 "Capacitors_SMD:CP_Elec_5x5.3" H 10750 1650 50  0001 C CNN
+F 3 "~" H 10750 1650 50  0001 C CNN
+	1    10750 1650
+	1    0    0    -1
+$EndComp
+Wire Wire Line
+	10750 1550 10750 1350
+Wire Wire Line
+	10750 1350 9800 1350
+Wire Wire Line
+	9800 1550 9900 1550
+Wire Wire Line
+	9900 1550 10000 1550
+Connection ~ 9900 1550
+Connection ~ 10750 1550
+Connection ~ 10400 1550
+Wire Wire Line
+	10400 1550 10750 1550
+$Comp
+L power:GND #PWR0137
+U 1 1 5BA471A1
+P 9900 1850
+F 0 "#PWR0137" H 9900 1600 50  0001 C CNN
+F 1 "GND" H 9905 1677 50  0000 C CNN
+F 2 "" H 9900 1850 50  0001 C CNN
+F 3 "" H 9900 1850 50  0001 C CNN
+	1    9900 1850
+	1    0    0    -1
+$EndComp
+Wire Notes Line
+	11150 600  11150 2200
+Wire Notes Line
+	600  600  11150 600
+Wire Notes Line
+	600  2200 11150 2200
+Wire Notes Line
+	6850 600  6850 2200
+Text Notes 9250 750  0    50   ~ 0
+5V\n
+$Comp
+L power:+5V #PWR0138
+U 1 1 5BA4A57D
+P 10750 1350
+F 0 "#PWR0138" H 10750 1200 50  0001 C CNN
+F 1 "+5V" H 10765 1523 50  0000 C CNN
+F 2 "" H 10750 1350 50  0001 C CNN
+F 3 "" H 10750 1350 50  0001 C CNN
+	1    10750 1350
+	1    0    0    -1
+$EndComp
+Connection ~ 10750 1350
+Wire Wire Line
+	10300 1550 10400 1550
+Wire Wire Line
+	4000 1200 4400 1200
 $EndSCHEMATC

Commit message: added esp and rfm
Parts:
- removed D2: 1N4001, Diodes_SMD:D_SMA, symbol Diode:1N4001
- added C1, C13: 100n, Capacitors_SMD:C_0603, symbol Device:C_Small
- added J5: Ant, Connectors_Molex:Molex_SMA_Jack_Edge_Mount, symbol Connector:Conn_Coaxial
- added R10, R11, R12, R13, R14: 10k, Resistors_SMD:R_0603, symbol Device:R_Small
- added SW1: Flash, Buttons_Switches_SMD:SW_DIP_x1_W5.08mm_Slide_Copal_CHS-A, symbol Switch:SW_Push
- added SW2: Reset, Buttons_Switches_SMD:SW_DIP_x1_W5.08mm_Slide_Copal_CHS-A, symbol Switch:SW_Push
- added U3: RFM69HCW, RF_Modules:HOPERF-RFM69HW, symbol RF_AM_FM:RFM69HCW
- added U4: ESP-12E, RF_Modules:ESP-12E, symbol RF_Module:ESP-12E
Connections:
- net labels added: ANT, GPIO0, GPIO4, GPIO5, MISO, MOSI, NSS, RESET, RXD_ESP, SCK, TXD_ESP
- wire segments 53 -> 61

Commit message: added programming header
Parts:
- added J8: Conn_01x05_Male, Pin_Headers:Pin_Header_Straight_1x05_Pitch2.54mm, symbol Connector:Conn_01x05_Male
Changed lines of the file:
@@
 L power:VCC #PWR0147
 U 1 1 5BA6515E
-P 6250 4300
-F 0 "#PWR0147" H 6250 4150 50  0001 C CNN
-F 1 "VCC" H 6267 4473 50  0000 C CNN
-F 2 "" H 6250 4300 50  0001 C CNN
-F 3 "" H 6250 4300 50  0001 C CNN
-	1    6250 4300
-	1    0    0    -1
+P 7250 5000
+F 0 "#PWR0147" H 7250 4850 50  0001 C CNN
+F 1 "VCC" H 7267 5173 50  0000 C CNN
+F 2 "" H 7250 5000 50  0001 C CNN
+F 3 "" H 7250 5000 50  0001 C CNN
+	1    7250 5000
+	0    1    1    0
 $EndComp
 Wire Wire Line
@@
 	1    0    0    -1
 $EndComp
+$Comp
+L Connector:Conn_01x05_Male J8
+U 1 1 5BA8C2CF
+P 7050 4800
+F 0 "J8" H 7156 5178 50  0000 C CNN
+F 1 "Conn_01x05_Male" H 7156 5087 50  0000 C CNN
+F 2 "Pin_Headers:Pin_Header_Straight_1x05_Pitch2.54mm" H 7050 4800 50  0001 C CNN
+F 3 "~" H 7050 4800 50  0001 C CNN
+	1    7050 4800
+	1    0    0    -1
+$EndComp
+$Comp
+L power:GND #PWR0104
+U 1 1 5BA8C5F5
+P 7250 4900
+F 0 "#PWR0104" H 7250 4650 50  0001 C CNN
+F 1 "GND" H 7100 4850 50  0000 C CNN
+F 2 "" H 7250 4900 50  0001 C CNN
+F 3 "" H 7250 4900 50  0001 C CNN
+	1    7250 4900
+	0    -1   -1   0
+$EndComp
+Text GLabel 7250 4800 2    50   Input ~ 0
+GPIO5
+Text GLabel 7250 4600 2    50   Input ~ 0
+TXD_ESP
+Text GLabel 7250 4700 2    50   Input ~ 0
+RXD_ESP
 $EndSCHEMATC

Commit message: moved libraries
Parts:
- removed J5: Ant, Connectors_Molex:Molex_SMA_Jack_Edge_Mount, symbol Connector:Conn_Coaxial
- added AE1: Antenna_Loop, otter:868MHZ Inverted-F, symbol Device:Antenna_Loop
- added C14: C_Small, Capacitor_SMD:C_0603_1608Metric, symbol Device:C_Small
- C1, C10, C11, C13, C2, C3, C5, C6, C7, C8: footprint Capacitors_SMD:C_0603 -> Capacitor_SMD:C_0603_1608Metric
- C12, C9: footprint Capacitors_SMD:CP_Elec_5x5.3 -> Capacitor_SMD:CP_Elec_5x5.3
- C4: footprint Capacitors_SMD:C_0805 -> Capacitor_SMD:C_0805_2012Metric
- D1, D4: footprint Diodes_SMD:D_SMA -> Diode_SMD:D_SMA
- D3: footprint LEDs:LED_0805 -> LED_SMD:LED_0805_2012Metric
- J1, J2: footprint Connectors_JST:JST_XH_B04B-XH-A_04x2.50mm_Straight -> Connector_JST:JST_XH_B04B-XH-A_1x04_P2.50mm_Vertical
- J3, J4, J6: footprint Pin_Headers:Pin_Header_Angled_1x04_Pitch2.54mm -> Connector_PinHeader_2.54mm:PinHeader_1x04_P2.54mm_Horizontal
- J7: footprint Pin_Headers:Pin_Header_Angled_1x02_Pitch2.54mm -> Connector_PinHeader_2.54mm:PinHeader_1x02_P2.54mm_Horizontal
- J8: footprint Pin_Headers:Pin_Header_Straight_1x05_Pitch2.54mm -> Connector_PinHeader_2.54mm:PinHeader_1x05_P2.54mm_Vertical
- L1: footprint Inductors_SMD:L_Taiyo-Yuden_MD-5050 -> Inductor_SMD:L_Taiyo-Yuden_MD-5050
- MH1, MH2, MH3, MH4: footprint Mounting_Holes:MountingHole_3.2mm_M3 -> MountingHole:MountingHole_3.2mm_M3
- R1, R10, R11, R12, R13, R14, R2, R3, R4, R5, R6, R7, R8, R9: footprint Resistors_SMD:R_0603 -> Resistor_SMD:R_0603_1608Metric
- SW1, SW2: footprint Buttons_Switches_SMD:SW_DIP_x1_W5.08mm_Slide_Copal_CHS-A -> Button_Switch_SMD:SW_DIP_SPSTx01_Slide_Copal_CHS-01A_W5.08mm_P1.27mm_JPin
- U1: footprint TO_SOT_Packages_SMD:SOT-223-3_TabPin2 -> Package_TO_SOT_SMD:SOT-223-3_TabPin2
- U2: footprint TO_SOT_Packages_SMD:TO-263-5_TabPin3 -> Package_TO_SOT_SMD:TO-263-5_TabPin3
- U3: footprint RF_Modules:HOPERF-RFM69HW -> RF_Module:HOPERF_RFM69HW
- U4: footprint RF_Modules:ESP-12E -> RF_Module:ESP-12E
Connections:
- wire segments 61 -> 63

Commit message: v1 finished
Parts:
- removed AE1: Antenna_Loop, otter:868MHZ Inverted-F, symbol Device:Antenna_Loop
- removed J7: VCC, Connector_PinHeader_2.54mm:PinHeader_1x02_P2.54mm_Horizontal, symbol Connector:Conn_01x02_Male
- added AE1: Antenna, Connector_Pin:Pin_D1.0mm_L10.0mm, symbol Device:Antenna
- added J5: Power, Connector_PinHeader_2.54mm:PinHeader_1x03_P2.54mm_Horizontal, symbol Connector:Conn_01x03_Male
Connections:
- wire segments 63 -> 64
Other:
- moved on the sheet: U3

Commit message: minor changes, now v2
Parts:
- removed C11: 100n, Capacitor_SMD:C_0603_1608Metric, symbol Device:C_Small
- removed D1: 1N4001, Diode_SMD:D_SMA, symbol Diode:1N4001
- removed D4: 1N5822, Diode_SMD:D_SMA, symbol Diode:1N5822
- removed J5: Power, Connector_PinHeader_2.54mm:PinHeader_1x03_P2.54mm_Horizontal, symbol Connector:Conn_01x03_Male
- removed J6: Nunchuk, Connector_PinHeader_2.54mm:PinHeader_1x04_P2.54mm_Horizontal, symbol Connector:Conn_01x04_Male
- removed L1: L, Inductor_SMD:L_Taiyo-Yuden_MD-5050, symbol Device:L
- removed U2: LM2596S-5, Package_TO_SOT_SMD:TO-263-5_TabPin3, symbol Regulator_Switching:LM2596S-5
- added D1: 12V, Diode_SMD:D_SMB, symbol Device:D_Zener
- added J7: xt30, otter:XT60_angle, symbol Connector:Conn_01x02_Male
- added J9: Conn_01x16_Female, Connector_PinHeader_2.54mm:PinHeader_1x16_P2.54mm_Vertical, symbol Connector:Conn_01x16_Female
- added P1: CONN_WII, otter:CONN_WII, symbol otter:CONN_WII
- added Q1: Q_NMOS_GDS, Package_TO_SOT_SMD:SOT-23, symbol Device:Q_NMOS_GDS
- added Q2: Q_PMOS_GDS, Package_TO_SOT_SMD:TO-252-2, symbol Device:Q_PMOS_GDS
- added R15, R16, R17: 100k, Resistor_SMD:R_0603_1608Metric, symbol Device:R_Small
- added R18, R19, R20, R27, R28: 10k, Resistor_SMD:R_0603_1608Metric, symbol Device:R_Small
- added R21, R22, R23: DNP, Resistor_SMD:R_0603_1608Metric, symbol Device:R_Small
- added R26: 220, Resistor_SMD:R_0603_1608Metric, symbol Device:R_Small
- added U2: URB4805YMD-6WR3, otter:URB4805YMD-6WR3, symbol otter:URB4805YMD-6WR3
- added U5: PCF8574, Package_SO:SOIC-16W_7.5x10.3mm_P1.27mm, symbol Interface_Expansion:PCF8574
- C12, C9: value 470u -> 20u
- J3: value Display -> Conn_01x04_Male; footprint Connector_PinHeader_2.54mm:PinHeader_1x04_P2.54mm_Horizontal -> Connector_PinHeader_2.54mm:PinHeader_1x04_P2.54mm_Vertical
- J4: footprint Connector_PinHeader_2.54mm:PinHeader_1x04_P2.54mm_Horizontal -> Connector_PinHeader_2.54mm:PinHeader_1x04_P2.54mm_Vertical
Connections:
- net labels added: A0, A1, A2, CS, DB4, DB5, DB6, DB7, LED_K, P3, RS, RW, VO, WS2812
- wire segments 64 -> 85
Other:
- note removed: "Display"

Commit message: minor changes
Changed lines of the file:
@@
 L Device:R R4
 U 1 1 5BA3D05F
-P 1600 1000
-F 0 "R4" V 1450 1000 50  0000 C CNN
-F 1 "1k" V 1600 1000 50  0000 C CNN
-F 2 "Resistor_SMD:R_0603_1608Metric" V 1530 1000 50  0001 C CNN
-F 3 "~" H 1600 1000 50  0001 C CNN
-	1    1600 1000
+P 2150 1000
+F 0 "R4" V 2000 1000 50  0000 C CNN
+F 1 "1k" V 2150 1000 50  0000 C CNN
+F 2 "Resistor_SMD:R_0603_1608Metric" V 2080 1000 50  0001 C CNN
+F 3 "~" H 2150 1000 50  0001 C CNN
+	1    2150 1000
 	0    1    1    0
 $EndComp
@@
 L Device:R R5
 U 1 1 5BA3D114
-P 1600 1100
-F 0 "R5" V 1700 1100 50  0000 C CNN
-F 1 "1k" V 1600 1100 50  0000 C CNN
-F 2 "Resistor_SMD:R_0603_1608Metric" V 1530 1100 50  0001 C CNN
-F 3 "~" H 1600 1100 50  0001 C CNN
-	1    1600 1100
+P 2150 1100
+F 0 "R5" V 2250 1100 50  0000 C CNN
+F 1 "1k" V 2150 1100 50  0000 C CNN
+F 2 "Resistor_SMD:R_0603_1608Metric" V 2080 1100 50  0001 C CNN
+F 3 "~" H 2150 1100 50  0001 C CNN
+	1    2150 1100
 	0    1    1    0
 $EndComp
@@
 L Device:R R6
 U 1 1 5BA3D17D
-P 1600 1650
-F 0 "R6" V 1450 1650 50  0000 C CNN
-F 1 "1k" V 1600 1650 50  0000 C CNN
-F 2 "Resistor_SMD:R_0603_1608Metric" V 1530 1650 50  0001 C CNN
-F 3 "~" H 1600 1650 50  0001 C CNN
-	1    1600 1650
+P 2200 1650
+F 0 "R6" V 2050 1650 50  0000 C CNN
+F 1 "1k" V 2200 1650 50  0000 C CNN
+F 2 "Resistor_SMD:R_0603_1608Metric" V 2130 1650 50  0001 C CNN
+F 3 "~" H 2200 1650 50  0001 C CNN
+	1    2200 1650
 	0    1    1    0
 $EndComp
@@
 L Device:R R7
 U 1 1 5BA3D1EC
-P 1600 1750
-F 0 "R7" V 1700 1750 50  0000 C CNN
-F 1 "1k" V 1600 1750 50  0000 C CNN
-F 2 "Resistor_SMD:R_0603_1608Metric" V 1530 1750 50  0001 C CNN
-F 3 "~" H 1600 1750 50  0001 C CNN
-	1    1600 1750
+P 2200 1750
+F 0 "R7" V 2300 1750 50  0000 C CNN
+F 1 "1k" V 2200 1750 50  0000 C CNN
+F 2 "Resistor_SMD:R_0603_1608Metric" V 2130 1750 50  0001 C CNN
+F 3 "~" H 2200 1750 50  0001 C CNN
+	1    2200 1750
 	0    1    1    0
 $EndComp
 Wire Wire Line
-	1100 1650 1450 1650
-Wire Wire Line
-	1100 1750 1450 1750
-Wire Wire Line
-	1750 1750 2200 1750
-Wire Wire Line
-	2400 1650 1850 1650
-Wire Wire Line
 	1100 900  2400 900
-Wire Wire Line
-	1100 1000 1450 1000
-Wire Wire Line
-	1100 1100 1450 1100
-Wire Wire Line
-	1750 1100 2200 1100
-Wire Wire Line
-	2400 1000 1850 1000
 $Comp
 L Device:C_Small C5
 U 1 1 5BA3F1C0
-P 1850 1250
-F 0 "C5" H 1942 1296 50  0000 L CNN
-F 1 "10n" H 1942 1205 50  0000 L CNN
-F 2 "Capacitor_SMD:C_0603_1608Metric" H 1850 1250 50  0001 C CNN
-F 3 "~" H 1850 1250 50  0001 C CNN
-	1    1850 1250
+P 1550 1250
+F 0 "C5" H 1642 1296 50  0000 L CNN
+F 1 "10n" H 1642 1205 50  0000 L CNN
+F 2 "Capacitor_SMD:C_0603_1608Metric" H 1550 1250 50  0001 C CNN
+F 3 "~" H 1550 1250 50  0001 C CNN
+	1    1550 1250
 	1    0    0    -1
 $EndComp
@@
 L Device:C_Small C7
 U 1 1 5BA3F21E
-P 2200 1250
-F 0 "C7" H 2292 1296 50  0000 L CNN
-F 1 "10n" H 2292 1205 50  0000 L CNN
-F 2 "Capacitor_SMD:C_0603_1608Metric" H 2200 1250 50  0001 C CNN
-F 3 "~" H 2200 1250 50  0001 C CNN
-	1    2200 1250
+P 1900 1250
+F 0 "C7" H 1992 1296 50  0000 L CNN
+F 1 "10n" H 1992 1205 50  0000 L CNN
+F 2 "Capacitor_SMD:C_0603_1608Metric" H 1900 1250 50  0001 C CNN
+F 3 "~" H 1900 1250 50  0001 C CNN
+	1    1900 1250
 	1    0    0    -1
 $EndComp
@@
 L Device:C_Small C6
 U 1 1 5BA3F287
-P 1850 1900
-F 0 "C6" H 1942 1946 50  0000 L CNN
-F 1 "10n" H 1942 1855 50  0000 L CNN
-F 2 "Capacitor_SMD:C_0603_1608Metric" H 1850 1900 50  0001 C CNN
-F 3 "~" H 1850 1900 50  0001 C CNN
-	1    1850 1900
+P 1550 1900
+F 0 "C6" H 1642 1946 50  0000 L CNN
+F 1 "10n" H 1642 1855 50  0000 L CNN
+F 2 "Capacitor_SMD:C_0603_1608Metric" H 1550 1900 50  0001 C CNN
+F 3 "~" H 1550 1900 50  0001 C CNN
+	1    1550 1900
 	1    0    0    -1
 $EndComp
@@
 L Device:C_Small C8
 U 1 1 5BA3F2EB
-P 2200 1900
-F 0 "C8" H 2292 1946 50  0000 L CNN
-F 1 "10n" H 2292 1855 50  0000 L CNN
-F 2 "Capacitor_SMD:C_0603_1608Metric" H 2200 1900 50  0001 C CNN
-F 3 "~" H 2200 1900 50  0001 C CNN
-	1    2200 1900
+P 1900 1900
+F 0 "C8" H 1992 1946 50  0000 L CNN
+F 1 "10n" H 1992 1855 50  0000 L CNN
+F 2 "Capacitor_SMD:C_0603_1608Metric" H 1900 1900 50  0001 C CNN
+F 3 "~" H 1900 1900 50  0001 C CNN
+	1    1900 1900
 	1    0    0    -1
 $EndComp
@@
 L power:GND #PWR0116
 U 1 1 5BA3F3C4
-P 1850 1350
-F 0 "#PWR0116" H 1850 1100 50  0001 C CNN
-F 1 "GND" H 1850 1200 50  0000 C CNN
-F 2 "" H 1850 1350 50  0001 C CNN
-F 3 "" H 1850 1350 50  0001 C CNN
-	1    1850 1350
+P 1550 1350
+F 0 "#PWR0116" H 1550 1100 50  0001 C CNN
+F 1 "GND" H 1550 1200 50  0000 C CNN
+F 2 "" H 1550 1350 50  0001 C CNN
+F 3 "" H 1550 1350 50  0001 C CNN
+	1    1550 1350
 	1    0    0    -1
 $EndComp
@@
 L power:GND #PWR0117
 U 1 1 5BA3F425
-P 2200 1350
-F 0 "#PWR0117" H 2200 1100 50  0001 C CNN
-F 1 "GND" H 2200 1200 50  0000 C CNN
-F 2 "" H 2200 1350 50  0001 C CNN
-F 3 "" H 2200 1350 50  0001 C CNN
-	1    2200 1350
+P 1900 1350
+F 0 "#PWR0117" H 1900 1100 50  0001 C CNN
+F 1 "GND" H 1900 1200 50  0000 C CNN
+F 2 "" H 1900 1350 50  0001 C CNN
+F 3 "" H 1900 1350 50  0001 C CNN
+	1    1900 1350
 	1    0    0    -1
 $EndComp
@@
 L power:GND #PWR0118
 U 1 1 5BA3F486
-P 1850 2000
-F 0 "#PWR0118" H 1850 1750 50  0001 C CNN
-F 1 "GND" H 1850 1850 50  0000 C CNN
-F 2 "" H 1850 2000 50  0001 C CNN
-F 3 "" H 1850 2000 50  0001 C CNN
-	1    1850 2000
+P 1550 2000
+F 0 "#PWR0118" H 1550 1750 50  0001 C CNN
+F 1 "GND" H 1550 1850 50  0000 C CNN
+F 2 "" H 1550 2000 50  0001 C CNN
+F 3 "" H 1550 2000 50  0001 C CNN
+	1    1550 2000
 	1    0    0    -1
 $EndComp
@@
 L power:GND #PWR0119
 U 1 1 5BA3F4E7
-P 2200 2000
-F 0 "#PWR0119" H 2200 1750 50  0001 C CNN
-F 1 "GND" H 2200 1850 50  0000 C CNN
-F 2 "" H 2200 2000 50  0001 C CNN
-F 3 "" H 2200 2000 50  0001 C CNN
-	1    2200 2000
-	1    0    0    -1
-$EndComp
-Wire Wire Line
-	1850 1800 1850 1650
-Connection ~ 1850 1650
-Wire Wire Line
-	1850 1650 1750 1650
-Wire Wire Line
-	2200 1800 2200 1750
-Connection ~ 2200 1750
-Wire Wire Line
-	2200 1750 2400 1750
-Wire Wire Line
-	2200 1150 2200 1100
-Connection ~ 2200 1100
-Wire Wire Line
-	2200 1100 2400 1100
-Wire Wire Line
-	1850 1150 1850 1000
-Connection ~ 1850 1000
-Wire Wire Line
-	1850 1000 1750 1000
+P 1900 2000
+F 0 "#PWR0119" H 1900 1750 50  0001 C CNN
+F 1 "GND" H 1900 1850 50  0000 C CNN
+F 2 "" H 1900 2000 50  0001 C CNN
+F 3 "" H 1900 2000 50  0001 C CNN
+	1    1900 2000
+	1    0    0    -1
+$EndComp
+Wire Wire Line
+	1550 1800 1550 1650
+Wire Wire Line
+	1900 1800 1900 1750
+Wire Wire Line
+	1900 1150 1900 1100
+Wire Wire Line
+	1550 1150 1550 1000
 Text Notes 1800 700  0    50   ~ 0
 Input
@@
 Wire Notes Line
 	3850 5150 3850 5850
+Wire Wire Line
+	2300 1000 2400 1000
+Wire Wire Line
+	2400 1100 2300 1100
+Wire Wire Line
+	1100 1000 1550 1000
+Wire Wire Line
+	1100 1100 1900 1100
+Connection ~ 1550 1000
+Wire Wire Line
+	1550 1000 2000 1000
+Connection ~ 1900 1100
+Wire Wire Line
+	1900 1100 2000 1100
+Wire Wire Line
+	2350 1650 2400 1650
+Wire Wire Line
+	2400 1750 2350 1750
+Wire Wire Line
+	1100 1750 1900 1750
+Wire Wire Line
+	1100 1650 1550 1650
+Connection ~ 1550 1650
+Wire Wire Line
+	1550 1650 2050 1650
+Connection ~ 1900 1750
+Wire Wire Line
+	1900 1750 2050 1750
 $EndSCHEMATC
